File: kosmo_proto/kosmo_proto.sch (KiCad schematic (older format))
At the start: 11 parts, among them J9901 Conn_01x01, J9902 Conn_01x01, J9903 Conn_01x01, J9904 Conn_01x01, J9905 Conn_01x01, J9906 Conn_01x01, J9907 EURO_PWR_2x5

Commit message: Replace fuses with diodes; improve layout; add row/column identifiers
Parts:
- removed F9901, F9902: RXEF025, ao_tht:PPTC_RXEF025, symbol Device:Polyfuse
- removed J9907: EURO_PWR_2x5, ao_tht:Power_Header, symbol kosmo_proto:Synth_power_2x5
- added D1, D2: 1N5817, ao_tht:D_DO-41_SOD81_P7.62mm_Horizontal, symbol Diode:1N5817
- added J1: Synth_power_2x5, ao_tht:Power_Header, symbol ao_symbols:Synth_power_2x5
- renumbered C9901 to C1, C9902 to C2, J9901 to J2, J9904 to J3, J9902 to J4, J9905 to J5, J9903 to J6, J9906 to J7
Other:
- moved on the sheet: C1, C2, J2, J3, J4, J5, J6, J7

Commit message: Dupe numbers and letters; add text/logo; change cap footprints; size and positioning tweaks
Parts:
- added GRAF1: AO logo, ao_tht:analogoutput_12mm, symbol ao_symbols:Graphic
- added GRAF2: CC0 logo, ao_tht:CC0_logo, symbol ao_symbols:Graphic
- C1, C2: footprint ao_tht:CP_Radial_D5.0mm_P2.00mm -> ao_tht:CP_Radial_D6.3mm_P2.50mm
Changed lines of the file:
@@
 F 0 "C1" H 5418 2296 50  0000 L CNN
 F 1 "10uF" H 5418 2205 50  0000 L CNN
-F 2 "ao_tht:CP_Radial_D5.0mm_P2.00mm" H 5338 2100 50  0001 C CNN
+F 2 "ao_tht:CP_Radial_D6.3mm_P2.50mm" H 5338 2100 50  0001 C CNN
 F 3 "~" H 5300 2250 50  0001 C CNN
 	1    5300 2250
@@
 F 0 "C2" H 5418 2596 50  0000 L CNN
 F 1 "10uF" H 5418 2505 50  0000 L CNN
-F 2 "ao_tht:CP_Radial_D5.0mm_P2.00mm" H 5338 2400 50  0001 C CNN
+F 2 "ao_tht:CP_Radial_D6.3mm_P2.50mm" H 5338 2400 50  0001 C CNN
 F 3 "~" H 5300 2550 50  0001 C CNN
 	1    5300 2550
@@
 	-1   0    0    1
 $EndComp
+$Comp
+L ao_symbols:Graphic GRAF1
+U 1 1 608D0242
+P 3300 3500
+F 0 "GRAF1" H 3578 3546 50  0000 L CNN
+F 1 "AO logo" H 3578 3455 50  0000 L CNN
+F 2 "ao_tht:analogoutput_12mm" H 3300 3500 50  0001 C CNN
+F 3 "" H 3300 3500 50  0001 C CNN
+F 4 "DNF" H 3300 3500 50  0001 C CNN "Config"
+	1    3300 3500
+	1    0    0    -1
+$EndComp
+$Comp
+L ao_symbols:Graphic GRAF2
+U 1 1 608D4A4C
+P 3300 3800
+F 0 "GRAF2" H 3578 3846 50  0000 L CNN
+F 1 "CC0 logo" H 3578 3755 50  0000 L CNN
+F 2 "ao_tht:CC0_logo" H 3300 3800 50  0001 C CNN
+F 3 "" H 3300 3800 50  0001 C CNN
+F 4 "DNF" H 3300 3800 50  0001 C CNN "Config"
+	1    3300 3800
+	1    0    0    -1
+$EndComp
 $EndSCHEMATC
